File: KiCad/BSPD v4 Rev 5.kicad_pcb (KiCad board)
At the start: 4 copper layers, 100 x 77.5 mm, 201 parts, among them J1 DTM13-12PA, U1 LM339, U10 2N7002, U11 2N7002, U12 2N7002, U13 2N7002, U14 2N7002, U15 2N7002, U16 2N7002, U17 74HC08D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

Commit message: Fixed, swapped relay symbol swapped NC and NO (same wiring maintained)
Connections:
- J1 pad 10: Relay_NO -> Relay_NC
- J1 pad 11: Relay_NC -> Relay_NO
- U23 pad 3: Relay_NO -> Relay_NC
- U23 pad 4: Relay_NC -> Relay_NO
Changed lines of the file:
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@@
 			(layers "*.Cu" "*.Mask")
 			(remove_unused_layers no)
-			(net 22 "Relay_NO")
+			(net 23 "Relay_NC")
 			(pinfunction "10")
 			(pintype "passive")
@@
 			(layers "*.Cu" "*.Mask")
 			(remove_unused_layers no)
-			(net 23 "Relay_NC")
+			(net 22 "Relay_NO")
 			(pinfunction "11")
 			(pintype "passive")
@@
 			)
 		)
-		(property "Datasheet" "https://www.lcsc.com/product-detail/C5355536.html"
+		(property "Datasheet" "https://lcsc.com/product-detail/Automotive-Relays_PANASONIC-ACNM1112_C5355536.html"
 			(at 0 0 0)
 			(unlocked yes)
@@
 			(layers "*.Cu" "*.Mask")
 			(remove_unused_layers no)
-			(net 22 "Relay_NO")
-			(pinfunction "NO")
+			(net 23 "Relay_NC")
+			(pinfunction "NC")
 			(pintype "passive")
 		)
@@
 			(layers "*.Cu" "*.Mask")
 			(remove_unused_layers no)
-			(net 23 "Relay_NC")
-			(pinfunction "NC")
+			(net 22 "Relay_NO")
+			(pinfunction "NO")
 			(pintype "passive")
 		)
@@
 	)
 	(segment
-		(start 156 138.75)
-		(end 174.7 138.75)
+		(start 154.25 133.75)
+		(end 154.25 102.56)
 		(width 1)
 		(layer "In1.Cu")
@@
 	)
 	(segment
-		(start 149.4 106.4)
-		(end 151.65 104.15)
+		(start 157 136.5)
+		(end 174.45 136.5)
 		(width 1)
 		(layer "In1.Cu")
@@
 	)
 	(segment
-		(start 174.7 138.75)
-		(end 177.45 141.5)
+		(start 157 136.5)
+		(end 154.25 133.75)
 		(width 1)
 		(layer "In1.Cu")
@@
 	)
 	(segment
-		(start 149.4 132.15)
-		(end 149.4 106.4)
+		(start 174.45 136.5)
+		(end 177.45 133.5)
 		(width 1)
 		(layer "In1.Cu")
@@
 	)
 	(segment
-		(start 156 138.75)
-		(end 149.4 132.15)
+		(start 154.25 102.56)
+		(end 151.65 99.96)
 		(width 1)
 		(layer "In1.Cu")
@@
 	)
 	(segment
-		(start 154.25 133.75)
-		(end 154.25 102.56)
+		(start 156 138.75)
+		(end 174.7 138.75)
 		(width 1)
 		(layer "In1.Cu")
@@
 	)
 	(segment
-		(start 157 136.5)
-		(end 174.45 136.5)
+		(start 149.4 106.4)
+		(end 151.65 104.15)
 		(width 1)
 		(layer "In1.Cu")
@@
 	)
 	(segment
-		(start 157 136.5)
-		(end 154.25 133.75)
+		(start 174.7 138.75)
+		(end 177.45 141.5)
 		(width 1)
 		(layer "In1.Cu")
@@
 	)
 	(segment
-		(start 174.45 136.5)
-		(end 177.45 133.5)
+		(start 149.4 132.15)
+		(end 149.4 106.4)
 		(width 1)
 		(layer "In1.Cu")
@@
 	)
 	(segment
-		(start 154.25 102.56)
-		(end 151.65 99.96)
+		(start 156 138.75)
+		(end 149.4 132.15)
 		(width 1)
 		(layer "In1.Cu")

Commit message: fixed fuckup
Connections:
- R10 pad 1: Net-(JP1-A) -> Net-(U2A--)
- R19 pad 2: Net-(U3B--) -> Net-(JP3-A)
- R20 pad 1: Net-(U3B--) -> Net-(JP3-A)
- R21 pad 2: Net-(JP3-A) -> Net-(U3C--)
- R22 pad 1: Net-(JP3-A) -> Net-(U3C--)
- R7 pad 2: Net-(U1D--) -> Net-(JP1-A)
- R8 pad 1: Net-(U1D--) -> Net-(JP1-A)
- R9 pad 2: Net-(JP1-A) -> Net-(U2A--)
- RV10 pad 2: Net-(U3B--) -> Net-(JP3-A)
- RV11 pad 2: Net-(JP3-A) -> Net-(U3C--)
- RV4 pad 2: Net-(U1D--) -> Net-(JP1-A)
- RV5 pad 2: Net-(JP1-A) -> Net-(U2A--)
- TP11 pad 1: Net-(JP3-A) -> Net-(U3C--)
- TP2 pad 1: Net-(U1D--) -> Net-(JP1-A)
- TP4 pad 1: Net-(U3B--) -> Net-(JP3-A)
- TP7 pad 1: Net-(JP1-A) -> Net-(U2A--)
- U1 pad 8: Net-(U1D--) -> Net-(JP2-C)
- U1 pad 9: TPS2 -> Net-(JP1-C)
- U2 pad 4: Net-(JP2-C) -> Net-(U2A--)
- U2 pad 5: Net-(JP1-C) -> TPS2
- U3 pad 10: Net-(JP4-C) -> Net-(U3C--)
- U3 pad 11: Net-(JP3-C) -> BRK2
- U3 pad 6: Net-(U3B--) -> Net-(JP4-C)
- U3 pad 7: BRK2 -> Net-(JP3-C)
Routing:
- net Net-(U3B--): track 161.9 -> 0.00 mm, vias 2 -> 0
- net Net-(U3C--): track 0.00 -> 149.4 mm, vias 0 -> 2
- net Net-(U2A--): track 0.00 -> 115.3 mm, vias 0 -> 2
- net Net-(U1D--): track 98.6 -> 0.00 mm, vias 3 -> 0
- net Net-(JP2-C): track 44.5 -> 12.3 mm
- net Net-(JP1-C): track 46.6 -> 21.5 mm
- net Net-(JP3-A): track 165.8 -> 183.0 mm
- net Net-(JP1-A): track 131.1 -> 123.4 mm, vias 1 -> 2
- net TPS2: track 88.0 -> 93.7 mm, vias 3 -> 2
- net BRK2: track 128.0 -> 123.8 mm, vias 3 -> 4
- net Net-(JP3-C): track 17.3 -> 20.7 mm
- net Net-(JP4-C): track 22.5 -> 21.0 mm
- net +5V: track 530.4 -> 531.9 mm
- net GND: vias 332 -> 331
